File: pcb/pcb.kicad_sch (KiCad schematic)
At the start: 249 parts, among them J1 USB_C_Receptacle_USB2.0, J2 AVR-ISP-6, SW1 1U, SW10 1U, SW100 ISO SHIFT, SW101 2U, SW102 1.25U CTRL, SW103 1.25U GUI, SW104 1.25U ALT, SW105 6.25u SPACE, SW106 1U ALT, SW107 1U GUI, SW108 1U CTRL, SW109 1U, SW11 1U, SW110 1U, SW111 1U, SW112 1U, SW113 1U, SW114 1U, SW115 1.5U CTRL, SW116 1U GUI, SW117 1.5U ALT, SW118 7U SPACE, SW119 1.5U ALT, SW12 1U, SW120 1.5U CTRL, SW121 1.5U GUI, SW122 6U SPACE, SW123 SW_Push, SW124 SW_Push, SW13 1U, SW14 1U, SW15 1U, SW16 1U, SW17 1U, SW18 1U, SW19 1U, SW2 1U, SW20 1U, SW21 1U, SW22 1U, SW23 1U, SW24 1U, SW25 1U, SW26 1U, SW27 1U, SW28 1U, SW29 1U, SW3 1U, SW30 1U, SW31 1U, SW32 1U, SW33 1U, SW34 1U, SW35 1U, SW36 1U, SW37 2U, SW38 1U, SW39 1U, SW4 1U, SW40 1U, SW41 1U, SW42 1U, SW43 1.5U, SW44 1U, SW45 1U, SW46 1U, SW47 1U, SW48 1U, SW49 1U, SW5 1U, SW50 1U, SW51 1U, SW52 1U, SW53 1U, SW54 1U, SW55 1U, SW56 1.5U, SW57 1U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

Commit message: Added 6U offset spacebar to PCB
Still need to add the cutout for the 6U offset spacebar switch to the switchplate.
Parts:
- added SW123: 6U OFF SPACE, Switch_Keyboard_Cherry_MX:SW_Cherry_MX_PCB_6.00u_Offset, symbol Switch:SW_Push
- SW122: footprint 0xcb:SW_Cherry_MX_PCB_3.00u -> Switch_Keyboard_Cherry_MX:SW_Cherry_MX_PCB_6.00u
- renumbered SW123 to SW124, SW124 to SW125
Connections:
- net COL3: now also SW123.2
- net at D98.2 (A), SW105.1, SW118.1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: now also SW123.1
Changed lines of the file:
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@@
   (junction (at 181.61 52.07) (diameter 0) (color 0 0 0 0)
   )
+  (junction (at 166.37 147.32) (diameter 0) (color 0 0 0 0)
+  )
   (junction (at 153.67 71.12) (diameter 0) (color 0 0 0 0)
   )
@@
   (junction (at 102.87 71.12) (diameter 0) (color 0 0 0 0)
   )
+  (junction (at 177.8 147.32) (diameter 0) (color 0 0 0 0)
+  )
   (junction (at 257.81 80.01) (diameter 0) (color 0 0 0 0)
   )
@@
     (stroke (width 0) (type default) (color 0 0 0 0))
   )
+  (wire (pts (xy 167.64 154.305) (xy 166.37 154.305))
+    (stroke (width 0) (type default) (color 0 0 0 0))
+  )
   (wire (pts (xy 102.87 114.3) (xy 102.87 127))
     (stroke (width 0) (type default) (color 0 0 0 0))
@@
     (stroke (width 0) (type default) (color 0 0 0 0))
   )
-  (wire (pts (xy 166.37 147.32) (xy 166.37 140.97))
-    (stroke (width 0) (type default) (color 0 0 0 0))
-  )
   (wire (pts (xy 306.07 85.09) (xy 306.07 99.06))
     (stroke (width 0) (type default) (color 0 0 0 0))
@@
     (stroke (width 0) (type default) (color 0 0 0 0))
   )
+  (wire (pts (xy 166.37 147.32) (xy 166.37 154.305))
+    (stroke (width 0) (type default) (color 0 0 0 0))
+  )
   (wire (pts (xy 255.27 113.03) (xy 255.27 127))
     (stroke (width 0) (type default) (color 0 0 0 0))
@@
     (stroke (width 0) (type default) (color 0 0 0 0))
   )
+  (wire (pts (xy 166.37 140.97) (xy 166.37 147.32))
+    (stroke (width 0) (type default) (color 0 0 0 0))
+  )
   (wire (pts (xy 156.21 50.8) (xy 156.21 52.07))
     (stroke (width 0) (type default) (color 0 0 0 0))
@@
     (stroke (width 0) (type default) (color 0 0 0 0))
   )
+  (wire (pts (xy 177.8 147.32) (xy 177.8 154.305))
+    (stroke (width 0) (type default) (color 0 0 0 0))
+  )
   (wire (pts (xy 229.87 43.18) (xy 229.87 71.12))
     (stroke (width 0) (type default) (color 0 0 0 0))
@@
       (effects (font (size 0.635 0.635)))
     )
-    (property "Footprint" "0xcb:SW_Cherry_MX_PCB_3.00u" (id 2) (at 171.45 142.24 0)
+    (property "Footprint" "Switch_Keyboard_Cherry_MX:SW_Cherry_MX_PCB_6.00u" (id 2) (at 171.45 142.24 0)
       (effects (font (size 1.27 1.27)) hide)
     )
@@
   (symbol (lib_id "Switch:SW_Push") (at 143.51 274.32 0) (unit 1)
     (in_bom yes) (on_board yes) (fields_autoplaced)
-    (property "Reference" "SW124" (id 0) (at 143.51 267.4325 0))
+    (property "Reference" "SW125" (id 0) (at 143.51 267.4325 0))
     (property "Value" "SW_Push" (id 1) (at 143.51 270.2076 0))
     (property "Footprint" "Button_Switch_THT:SW_PUSH_6mm_H5mm" (id 2) (at 143.51 269.24 0)
@@
     (pin "2")
   )
+  (symbol (lib_id "Switch:SW_Push") (at 172.72 154.305 0) (unit 1)
+    (in_bom yes) (on_board yes)
+    (property "Reference" "SW123" (id 0) (at 174.625 156.21 0))
+    (property "Value" "6U OFF SPACE" (id 1) (at 175.26 158.115 0)
+      (effects (font (size 0.635 0.635)))
+    )
+    (property "Footprint" "Switch_Keyboard_Cherry_MX:SW_Cherry_MX_PCB_6.00u_Offset" (id 2) (at 172.72 149.225 0)
+      (effects (font (size 1.27 1.27)) hide)
+    )
+    (property "Datasheet" "~" (id 3) (at 172.72 149.225 0)
+      (effects (font (size 1.27 1.27)) hide)
+    )
+    (pin "1")
+    (pin "2")
+  )
   (symbol (lib_id "Switch:SW_Push") (at 173.99 113.03 0) (unit 1)
     (in_bom yes) (on_board yes)
@@
   (symbol (lib_id "Switch:SW_Push") (at 113.03 270.51 0) (unit 1)
     (in_bom yes) (on_board yes) (fields_autoplaced)
-    (property "Reference" "SW123" (id 0) (at 113.03 263.6225 0))
+    (property "Reference" "SW124" (id 0) (at 113.03 263.6225 0))
     (property "Value" "SW_Push" (id 1) (at 113.03 266.3976 0))
     (property "Footprint" "Button_Switch_THT:SW_PUSH_6mm_H5mm" (id 2) (at 113.03 265.43 0)
@@
     )
     (path "/3d5d0f67-24dd-4ec0-a75c-164b57b95844"
-      (reference "SW122") (unit 1) (value "6U SPACE") (footprint "0xcb:SW_Cherry_MX_PCB_3.00u")
+      (reference "SW122") (unit 1) (value "6U SPACE") (footprint "Switch_Keyboard_Cherry_MX:SW_Cherry_MX_PCB_6.00u")
+    )
+    (path "/e6f7b6bb-e3ac-4fda-9477-f92398fc552a"
+      (reference "SW123") (unit 1) (value "6U OFF SPACE") (footprint "Switch_Keyboard_Cherry_MX:SW_Cherry_MX_PCB_6.00u_Offset")
     )
     (path "/fabae21c-0bf5-41e1-92c8-b0440c8cdf3c"
-      (reference "SW123") (unit 1) (value "SW_Push") (footprint "Button_Switch_THT:SW_PUSH_6mm_H5mm")
+      (reference "SW124") (unit 1) (value "SW_Push") (footprint "Button_Switch_THT:SW_PUSH_6mm_H5mm")
     )
     (path "/a7101267-ef19-45d2-8fa7-ae837c20a1af"
-      (reference "SW124") (unit 1) (value "SW_Push") (footprint "Button_Switch_THT:SW_PUSH_6mm_H5mm")
+      (reference "SW125") (unit 1) (value "SW_Push") (footprint "Button_Switch_THT:SW_PUSH_6mm_H5mm")
     )
     (path "/33c2894b-5bcb-4855-b7e6-bfea44f483a5"

Commit message: Updated 6u and 6u offset footprint to 0xCB
Parts:
- SW122: footprint Switch_Keyboard_Cherry_MX:SW_Cherry_MX_PCB_6.00u -> 0xcb:SW_Cherry_MX_PCB_6.00u
- SW123: footprint Switch_Keyboard_Cherry_MX:SW_Cherry_MX_PCB_6.00u_Offset -> 0xcb:SW_Cherry_MX_PCB_6.00u_offset
Changed lines of the file:
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@@
       (effects (font (size 0.635 0.635)))
     )
-    (property "Footprint" "Switch_Keyboard_Cherry_MX:SW_Cherry_MX_PCB_6.00u" (id 2) (at 171.45 142.24 0)
+    (property "Footprint" "0xcb:SW_Cherry_MX_PCB_6.00u" (id 2) (at 171.45 142.24 0)
       (effects (font (size 1.27 1.27)) hide)
     )
@@
       (effects (font (size 0.635 0.635)))
     )
-    (property "Footprint" "Switch_Keyboard_Cherry_MX:SW_Cherry_MX_PCB_6.00u_Offset" (id 2) (at 172.72 149.225 0)
+    (property "Footprint" "0xcb:SW_Cherry_MX_PCB_6.00u_offset" (id 2) (at 172.72 149.225 0)
       (effects (font (size 1.27 1.27)) hide)
     )
@@
     )
     (path "/3d5d0f67-24dd-4ec0-a75c-164b57b95844"
-      (reference "SW122") (unit 1) (value "6U SPACE") (footprint "Switch_Keyboard_Cherry_MX:SW_Cherry_MX_PCB_6.00u")
+      (reference "SW122") (unit 1) (value "6U SPACE") (footprint "0xcb:SW_Cherry_MX_PCB_6.00u")
     )
     (path "/e6f7b6bb-e3ac-4fda-9477-f92398fc552a"
-      (reference "SW123") (unit 1) (value "6U OFF SPACE") (footprint "Switch_Keyboard_Cherry_MX:SW_Cherry_MX_PCB_6.00u_Offset")
+      (reference "SW123") (unit 1) (value "6U OFF SPACE") (footprint "0xcb:SW_Cherry_MX_PCB_6.00u_offset")
     )
     (path "/fabae21c-0bf5-41e1-92c8-b0440c8cdf3c"
