File: switchplate/switchplate.kicad_pcb (KiCad board)
At the start: 2 copper layers, 381 x 144.9 mm, 0 parts

Commit message: Added copper fill to switchplate
Routing:
- net (no net): vias 0 -> 1
- added copper zone on B.Cu, net (none)
- added copper zone on F.Cu, net (none)
Changed lines of the file:
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@@
   (gr_line (start 302.4125 101.1) (end 315.4125 101.1) (layer "Edge.Cuts") (width 0.25))
   (gr_line (start 421.475 182.0625) (end 434.475 182.0625) (layer "Edge.Cuts") (width 0.25))
+  (via (at 388.9375 127) (size 0.8) (drill 0.4) (layers "F.Cu" "B.Cu") (free) (net 0))
+  (zone (net 0) (net_name "") (layers F&B.Cu) (hatch edge 0.508)
+    (connect_pads (clearance 0.508))
+    (min_thickness 0.254) (filled_areas_thickness no)
+    (fill yes (thermal_gap 0.508) (thermal_bridge_width 0.508))
+    (polygon
+      (pts
+        (xy 508 206.375)
+        (xy 119.0625 206.375)
+        (xy 119.0625 55.5625)
+        (xy 508 55.5625)
+      )
+    )
+  )
   (group "" (id c07eebcc-30d2-439d-8030-faea6ade4486)
     (members
