File: backplate/backplate.kicad_pcb (KiCad board)
At the start: 2 copper layers, 381 x 165.6 mm, 25 parts

Commit message: Moved top window support holes on backplate
Parts:
- moved MH2 2.38 mm to (470.7, 131.0)
- moved MH2 2.38 mm to (385.0, 131.0)
- moved MH2 2.38 mm to (107.2, 131.0)
- moved MH2 2.38 mm to (192.9, 131.0)
- moved MH2 1.59 mm to (385.0, 142.9)
- moved MH2 1.59 mm to (192.9, 142.9)
- moved MH2 1.59 mm to (107.2, 142.9)
- moved MH2 1.59 mm to (470.7, 142.9)
Changed lines of the file:
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@@
   )
   (footprint "0xcb:mount" (layer "F.Cu")
-    (at 470.69375 144.4625)
+    (at 470.69375 142.875)
     (attr exclude_from_pos_files exclude_from_bom)
     (fp_text reference "MH2" (at 0 2) (layer "Dwgs.User") hide
@@
   )
   (footprint "0xcb:mount" (layer "F.Cu")
-    (at 107.15625 133.35)
-    (attr exclude_from_pos_files exclude_from_bom)
-    (fp_text reference "MH2" (at 0 2) (layer "Dwgs.User") hide
-      (effects (font (size 1 1) (thickness 0.15)))
-    )
-    (fp_text value "Mount-M2" (at 0 -2) (layer "Dwgs.User") hide
-      (effects (font (size 1 1) (thickness 0.15)))
-    )
-    (pad "1" thru_hole circle (at 0 0) (size 3.500001 3.500001) (drill 2.2) (layers *.Cu *.Mask)
-      (net 1 "GND"))
-  )
-  (footprint "0xcb:mount" (layer "F.Cu")
-    (at 192.88125 133.35)
+    (at 107.15625 130.96875)
+    (attr exclude_from_pos_files exclude_from_bom)
+    (fp_text reference "MH2" (at 0 2) (layer "Dwgs.User") hide
+      (effects (font (size 1 1) (thickness 0.15)))
+    )
+    (fp_text value "Mount-M2" (at 0 -2) (layer "Dwgs.User") hide
+      (effects (font (size 1 1) (thickness 0.15)))
+    )
+    (pad "1" thru_hole circle (at 0 0) (size 3.500001 3.500001) (drill 2.2) (layers *.Cu *.Mask)
+      (net 1 "GND"))
+  )
+  (footprint "0xcb:mount" (layer "F.Cu")
+    (at 192.88125 130.96875)
     (attr exclude_from_pos_files exclude_from_bom)
     (fp_text reference "MH2" (at 0 2) (layer "Dwgs.User") hide
@@
   )
   (footprint "0xcb:mount" (layer "F.Cu")
-    (at 470.69375 133.35)
-    (attr exclude_from_pos_files exclude_from_bom)
-    (fp_text reference "MH2" (at 0 2) (layer "Dwgs.User") hide
-      (effects (font (size 1 1) (thickness 0.15)))
-    )
-    (fp_text value "Mount-M2" (at 0 -2) (layer "Dwgs.User") hide
-      (effects (font (size 1 1) (thickness 0.15)))
-    )
-    (pad "1" thru_hole circle (at 0 0) (size 3.500001 3.500001) (drill 2.2) (layers *.Cu *.Mask)
-      (net 1 "GND"))
-  )
-  (footprint "0xcb:mount" (layer "F.Cu")
-    (at 384.96875 133.35)
-    (attr exclude_from_pos_files exclude_from_bom)
-    (fp_text reference "MH2" (at 0 2) (layer "Dwgs.User") hide
-      (effects (font (size 1 1) (thickness 0.15)))
-    )
-    (fp_text value "Mount-M2" (at 0 -2) (layer "Dwgs.User") hide
-      (effects (font (size 1 1) (thickness 0.15)))
-    )
-    (pad "1" thru_hole circle (at 0 0) (size 3.500001 3.500001) (drill 2.2) (layers *.Cu *.Mask)
-      (net 1 "GND"))
-  )
-  (footprint "0xcb:mount" (layer "F.Cu")
-    (at 384.96875 144.4625)
+    (at 470.69375 130.96875)
+    (attr exclude_from_pos_files exclude_from_bom)
+    (fp_text reference "MH2" (at 0 2) (layer "Dwgs.User") hide
+      (effects (font (size 1 1) (thickness 0.15)))
+    )
+    (fp_text value "Mount-M2" (at 0 -2) (layer "Dwgs.User") hide
+      (effects (font (size 1 1) (thickness 0.15)))
+    )
+    (pad "1" thru_hole circle (at 0 0) (size 3.500001 3.500001) (drill 2.2) (layers *.Cu *.Mask)
+      (net 1 "GND"))
+  )
+  (footprint "0xcb:mount" (layer "F.Cu")
+    (at 384.96875 130.96875)
+    (attr exclude_from_pos_files exclude_from_bom)
+    (fp_text reference "MH2" (at 0 2) (layer "Dwgs.User") hide
+      (effects (font (size 1 1) (thickness 0.15)))
+    )
+    (fp_text value "Mount-M2" (at 0 -2) (layer "Dwgs.User") hide
+      (effects (font (size 1 1) (thickness 0.15)))
+    )
+    (pad "1" thru_hole circle (at 0 0) (size 3.500001 3.500001) (drill 2.2) (layers *.Cu *.Mask)
+      (net 1 "GND"))
+  )
+  (footprint "0xcb:mount" (layer "F.Cu")
+    (at 384.96875 142.875)
     (attr exclude_from_pos_files exclude_from_bom)
     (fp_text reference "MH2" (at 0 2) (layer "Dwgs.User") hide
@@
   )
   (footprint "0xcb:mount" (layer "F.Cu")
-    (at 192.88125 144.4625)
+    (at 192.88125 142.875)
     (attr exclude_from_pos_files exclude_from_bom)
     (fp_text reference "MH2" (at 0 2) (layer "Dwgs.User") hide
@@
   )
   (footprint "0xcb:mount" (layer "F.Cu")
-    (at 107.15625 144.4625)
+    (at 107.15625 142.875)
     (attr exclude_from_pos_files exclude_from_bom)
     (fp_text reference "MH2" (at 0 2) (layer "Dwgs.User") hide
@@
     (connect_pads (clearance 0.508))
     (min_thickness 0.254) (filled_areas_thickness no)
-    (fill yes (thermal_gap 0.508) (thermal_bridge_width 0.508))
+    (fill (thermal_gap 0.508) (thermal_bridge_width 0.508))
     (polygon
       (pts
