File: v0.2/pcb/pcb.kicad_pcb (KiCad board)
At the start: 2 copper layers, 381 x 165.6 mm, 261 parts, among them J1 USB_C_Receptacle_USB2.0, J2 AVR-ISP-6, SW1 1U, SW10 1U, SW100 1.25U GUI, SW101 1.25U ALT, SW102 1U, SW103 6.25u SPACE, SW104 1U ALT, SW105 1U GUI, SW106 1U CTRL, SW107 1U, SW108 1U, SW109 1U, SW11 1U, SW110 1U, SW111 1U, SW112 1U, SW113 1.5U CTRL, SW114 1.5U GUI, SW114 1U GUI, SW115 1.5U ALT, SW116 7U SPACE, SW117 1.5U ALT, SW118 1.5U CTRL, SW119 6U SPACE, SW12 1U, SW120 1U, SW121 1U, SW122 1U, SW123 6U OFF SPACE, SW124 10U SPACE, SW125 SW_Push, SW126 SW_Push, SW13 1U, SW14 1U, SW15 1U, SW16 1U, SW17 1U, SW18 1U, SW19 1U, SW2 1U, SW20 1U, SW21 1U, SW22 1U, SW23 1U, SW24 1U, SW25 1U, SW26 1U, SW27 1U, SW28 1U, SW29 1U, SW3 1U, SW30 1U, SW31 1U, SW32 1U, SW33 1U, SW34 1U, SW35 2U, SW36 1U, SW37 1U, SW38 1U, SW39 1U, SW4 1U, SW40 1.5U, SW41 1U, SW42 1U, SW43 1U, SW44 1U, SW45 1U, SW46 1U, SW47 1U, SW48 1U, SW49 1U, SW5 1U, SW50 1U, SW51 1U, SW52 1U, SW53 1.5U, SW54 1U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

Commit message: Updated schematic, add temp controller footprint
Parts:
- removed C1: 4.7u, Capacitor_THT:CP_Radial_D4.0mm_P1.50mm
- removed C2, C3: 0.1u, Capacitor_THT:C_Disc_D4.3mm_W1.9mm_P5.00mm
- removed C4, C5: 22p, Capacitor_THT:C_Disc_D3.0mm_W1.6mm_P2.50mm
- removed the D107 at (291.9, 141.3)
- removed D108: 3.6V, Diode_THT:D_DO-41_SOD81_P7.62mm_Horizontal
- removed the D96 at (289.6, 170.7)
- removed F1: 500mA, Fuse:Fuse_BelFuse_0ZRE0025FF_L9.6mm_W3.8mm
- removed J1: USB_C_Receptacle_USB2.0, Connector_USB:USB_C_Receptacle_GCT_USB4085
- removed J2: AVR-ISP-6, Connector_PinHeader_2.54mm:PinHeader_2x03_P2.54mm_Vertical
- removed R1, R3: 5.1K, Resistor_THT:R_Axial_DIN0204_L3.6mm_D1.6mm_P7.62mm_Horizontal
- removed R2: 1.5K, Resistor_THT:R_Axial_DIN0204_L3.6mm_D1.6mm_P7.62mm_Horizontal
- removed R4, R5: 75, Resistor_THT:R_Axial_DIN0204_L3.6mm_D1.6mm_P7.62mm_Horizontal
- removed R6: 10k, Resistor_THT:R_Axial_DIN0204_L3.6mm_D1.6mm_P7.62mm_Horizontal
- removed REF** (x6): Stabilizer_Cherry_MX_2u, 0xcb:Stabilizer_Cherry_MX_2u
- removed REF**: Stabilizer_Cherry_MX_8u, 0xcb:Stabilizer_Cherry_MX_8u
- removed REF**: Stabilizer_Cherry_MX_7u, 0xcb:Stabilizer_Cherry_MX_7u
- removed REF**: Stabilizer_Cherry_MX_6u, 0xcb:Stabilizer_Cherry_MX_6u
- removed REF**: Stabilizer_Cherry_MX_6.25u, 0xcb:Stabilizer_Cherry_MX_6.25u
- removed the SW102 at (169.9, 273.1)
- removed the SW114 at (141.3, 273.1)
- removed SW125, SW126: SW_Push, Button_Switch_THT:SW_PUSH_6mm_H5mm
- removed Y1: Crystal, Crystal:Crystal_HC49-4H_Vertical
- added D70: 1N4148, Diode_THT:D_DO-35_SOD27_P7.62mm_Horizontal, F.Cu at (343.7, 72.2)
- added D94: 1N4148, Diode_THT:D_DO-35_SOD27_P7.62mm_Horizontal, F.Cu at (295.4, 76.2)
- added SW103: 1U, 0xcb:SW_Cherry_MX_PCB_1.00u, F.Cu at (284.2, 273.1)
- SW102: renamed from SW103; value 6.25u SPACE -> 6.25U
- SW116: value 7U SPACE -> 7U
- SW122: renamed from SW119; value 6U SPACE -> 6U
- SW123: value 6U OFF SPACE -> 6U OFFSET
- SW124: value 10U SPACE -> 10U
- U1: value ATmega32A-P -> BlackPillSTM32F401-weact; footprint Package_DIP:DIP-40_W15.24mm -> BlackPill-STM32F401-temp:BlackPillSTM32F401CCU6
- moved U1 306.0 mm to (58.7, 162.7), turned to 90 degrees
- moved D14 99.2 mm to (295.4, 78.6)
- moved D18 99.2 mm to (318.1, 78.6)
- moved D28 99.2 mm to (172.9, 78.6)
- moved D31 99.2 mm to (150.2, 78.6)
- moved D39 99.2 mm to (322.4, 78.6)
- moved D46 99.2 mm to (199.9, 78.6)
- moved D51 99.2 mm to (177.2, 78.6)
- moved D54 99.2 mm to (345.1, 78.6)
- moved D64 99.2 mm to (226.9, 78.6)
- moved D69 99.2 mm to (204.2, 78.6)
- moved D75 99.2 mm to (349.4, 78.6)
- moved D77 99.2 mm to (231.1, 78.6)
- moved D8 99.2 mm to (123.2, 78.6)
- moved D82 99.2 mm to (264.2, 78.6)
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- renumbered D105 to D100, D106 to D101, D98 to D102, D100 to D103, D93 to D104, D94 to D105, D95 to D106, D97 to D107, D70 to D71, D71 to D72, D72 to D73, D73 to D74, D74 to D75, D75 to D76, D76 to D77, D77 to D78, D78 to D79, D79 to D80, D80 to D81, D81 to D82, D82 to D83, D83 to D84, D84 to D85, D85 to D86, D86 to D87, D87 to D88, D88 to D89, D89 to D90, D90 to D91, D91 to D92, D92 to D93, D99 to D95, D101 to D96, D102 to D97, D103 to D98, D104 to D99, SW120 to SW119, SW121 to SW120, SW122 to SW121, SW58 to SW40, SW40 to SW41, SW41 to SW42, SW42 to SW43, SW43 to SW44, SW44 to SW45, SW45 to SW46, SW46 to SW47, SW47 to SW48, SW48 to SW49, SW49 to SW50, SW50 to SW51, SW51 to SW52, SW52 to SW53, SW53 to SW54, SW54 to SW55, SW55 to SW56, SW56 to SW57, SW57 to SW58, SW78 to SW72, SW72 to SW73, SW73 to SW74, SW74 to SW75, SW75 to SW76, SW76 to SW77, SW77 to SW78, SW98 to SW80, SW97 to SW81, SW80 to SW82, SW81 to SW83, SW82 to SW84, SW83 to SW85, SW84 to SW86, SW85 to SW87, SW86 to SW88, SW87 to SW89, SW88 to SW90, SW89 to SW91, SW90 to SW92, SW91 to SW93, SW92 to SW94, SW93 to SW95, SW94 to SW96, SW95 to SW97, SW96 to SW98
Connections:
- D1 pad 1: ROW1 -> ROW0
- D100 pad 1: ROW11 -> ROW6
- D101 pad 1: ROW12 -> ROW6
- D102 pad 1: ROW12 -> ROW6
- D103 pad 1: ROW12 -> ROW6
- D104 pad 1: ROW12 -> ROW6
- D105 pad 1: ROW11 -> ROW6
- D106 pad 1: ROW12 -> ROW6
- D107 pad 1: ROW12 -> ROW6
- D11 pad 1: ROW1 -> ROW0
- D13 pad 1: ROW1 -> ROW0
- D15 pad 1: ROW1 -> ROW0
- D17 pad 1: ROW1 -> ROW0
- D18 pad 1: ROW2 -> ROW1
- D19 pad 1: ROW2 -> ROW1
- D20 pad 1: ROW2 -> ROW1
- D21 pad 1: ROW2 -> ROW1
- D22 pad 1: ROW4 -> ROW2
- D23 pad 1: ROW3 -> ROW2
- D24 pad 1: ROW4 -> ROW2
- D25 pad 1: ROW3 -> ROW2
- D26 pad 1: ROW4 -> ROW2
- D27 pad 1: ROW3 -> ROW2
- D28 pad 1: ROW4 -> ROW2
- D29 pad 1: ROW3 -> ROW2
- D3 pad 1: ROW1 -> ROW0
- D30 pad 1: ROW4 -> ROW2
- D31 pad 1: ROW3 -> ROW2
- D32 pad 1: ROW4 -> ROW2
- D33 pad 1: ROW3 -> ROW2
- D34 pad 1: ROW4 -> ROW2
- D35 pad 1: ROW3 -> ROW2
- D36 pad 1: ROW3 -> ROW2
- D37 pad 1: ROW4 -> ROW2
- D38 pad 1: ROW3 -> ROW2
- D39 pad 1: ROW4 -> ROW2
- D40 pad 1: ROW6 -> ROW3
- D41 pad 1: ROW5 -> ROW3
- D42 pad 1: ROW6 -> ROW3
- D43 pad 1: ROW5 -> ROW3
- D44 pad 1: ROW6 -> ROW3
- D45 pad 1: ROW5 -> ROW3
- D46 pad 1: ROW6 -> ROW3
- D47 pad 1: ROW5 -> ROW3
- D48 pad 1: ROW6 -> ROW3
- D49 pad 1: ROW5 -> ROW3
- D5 pad 1: ROW1 -> ROW0
- D50 pad 1: ROW6 -> ROW3
- D51 pad 1: ROW5 -> ROW3
- D52 pad 1: ROW6 -> ROW3
- D53 pad 1: ROW5 -> ROW3
- D54 pad 1: ROW5 -> ROW3
- D55 pad 1: ROW6 -> ROW3
- D56 pad 1: ROW5 -> ROW3
- D57 pad 1: ROW6 -> ROW3
- D58 pad 1: ROW8 -> ROW4
- D59 pad 1: ROW7 -> ROW4
- D60 pad 1: ROW8 -> ROW4
- D61 pad 1: ROW7 -> ROW4
- D62 pad 1: ROW8 -> ROW4
- D63 pad 1: ROW7 -> ROW4
- D64 pad 1: ROW8 -> ROW4
- D65 pad 1: ROW7 -> ROW4
- D66 pad 1: ROW8 -> ROW4
- D67 pad 1: ROW7 -> ROW4
- D68 pad 1: ROW8 -> ROW4
- D69 pad 1: ROW7 -> ROW4
- D7 pad 1: ROW1 -> ROW0
- D71 pad 1: ROW8 -> ROW4
- D72 pad 1: ROW7 -> ROW4
- D73 pad 1: ROW8 -> ROW4
- D74 pad 1: ROW7 -> ROW4
- D75 pad 1: ROW8 -> ROW4
- D76 pad 1: ROW10 -> ROW5
- D77 pad 1: ROW9 -> ROW5
- D78 pad 1: ROW10 -> ROW5
- D79 pad 1: ROW9 -> ROW5
- D80 pad 1: ROW10 -> ROW5
- D81 pad 1: ROW9 -> ROW5
- D82 pad 1: ROW10 -> ROW5
- D83 pad 1: ROW9 -> ROW5
- D84 pad 1: ROW10 -> ROW5
- D85 pad 1: ROW9 -> ROW5
- D86 pad 1: ROW10 -> ROW5
- D87 pad 1: ROW9 -> ROW5
- D88 pad 1: ROW10 -> ROW5
- D89 pad 1: ROW10 -> ROW5
- D9 pad 1: ROW1 -> ROW0
- D90 pad 1: ROW9 -> ROW5
- D91 pad 1: ROW10 -> ROW5
- D92 pad 1: ROW9 -> ROW5
- D93 pad 1: ROW10 -> ROW5
- D95 pad 1: ROW11 -> ROW6
- D96 pad 1: ROW11 -> ROW6
- D97 pad 1: ROW12 -> ROW6
- D98 pad 1: ROW11 -> ROW6
- D99 pad 1: ROW12 -> ROW6
- SW10 pad 2: COL4 -> COL9
- SW100 pad 2: COL0 -> COL1
- SW101 pad 2: COL1 -> COL2
- SW102 pad 2: COL3 -> COL6
- SW104 pad 2: COL5 -> COL9
- SW105 pad 2: COL5 -> COL10
- SW106 pad 2: COL6 -> COL11
- SW107 pad 2: COL6 -> unconnected-(SW107-Pad2)
- SW108 pad 2: COL7 -> COL13
- SW109 pad 2: COL7 -> COL14
- SW11 pad 2: COL5 -> COL10
- SW110 pad 2: COL8 -> COL15
- SW111 pad 2: COL8 -> COL16
- SW112 pad 2: COL9 -> COL17
- SW114 pad 2: COL0 -> COL1
- SW115 pad 2: COL1 -> COL2
- SW116 pad 2: COL3 -> COL6
- SW117 pad 2: COL5 -> COL9
- SW118 pad 2: COL6 -> COL11
- SW12 pad 2: COL5 -> COL11
- SW120 pad 2: COL0 -> COL1
- SW121 pad 2: COL1 -> COL2
- SW122 pad 2: COL3 -> COL6
- SW123 pad 2: COL3 -> COL6
- SW124 pad 2: COL3 -> COL6
- SW13 pad 2: COL6 -> COL12
- SW14 pad 2: COL7 -> COL14
- SW15 pad 2: COL8 -> COL15
- SW16 pad 2: COL8 -> COL16
- SW17 pad 2: COL9 -> COL17
- SW18 pad 2: COL6 -> COL14
- SW19 pad 2: COL7 -> COL15
- SW2 pad 2: COL0 -> COL1
- SW20 pad 2: COL8 -> COL16
- SW21 pad 2: COL9 -> COL17
- SW23 pad 2: COL0 -> COL1
- SW24 pad 2: COL1 -> COL2
- SW25 pad 2: COL1 -> COL3
- SW26 pad 2: COL2 -> COL4
- SW27 pad 2: COL2 -> COL5
- SW28 pad 2: COL3 -> COL6
- SW29 pad 2: COL3 -> COL7
- SW3 pad 2: COL1 -> COL2
- SW30 pad 2: COL4 -> COL8
- SW31 pad 2: COL4 -> COL9
- SW32 pad 2: COL5 -> COL10
- SW33 pad 2: COL5 -> COL11
- SW34 pad 2: COL6 -> COL12
- SW35 pad 2: COL6 -> COL13
- SW36 pad 2: COL7 -> COL14
- SW37 pad 2: COL8 -> COL15
- SW38 pad 2: COL8 -> COL16
- SW39 pad 2: COL9 -> COL17
- SW4 pad 2: COL1 -> COL3
- SW40 pad 2: COL9 -> COL17
- SW42 pad 2: COL0 -> COL1
- SW43 pad 2: COL1 -> COL2
- SW44 pad 2: COL1 -> COL3
- SW45 pad 2: COL2 -> COL4
- SW46 pad 2: COL2 -> COL5
- SW47 pad 2: COL3 -> COL6
- SW48 pad 2: COL3 -> COL7
- SW49 pad 2: COL4 -> COL8
- SW5 pad 2: COL2 -> COL4
- SW50 pad 2: COL4 -> COL9
- SW51 pad 2: COL5 -> COL10
- SW52 pad 2: COL5 -> COL11
- SW53 pad 2: COL6 -> COL12
- SW54 pad 2: COL6 -> COL13
- SW55 pad 2: COL7 -> COL14
- SW56 pad 2: COL8 -> COL15
- SW57 pad 2: COL8 -> COL16
- SW58 pad 2: COL9 -> COL17
- SW59 pad 2: COL6 -> COL13
- SW6 pad 2: COL2 -> COL5
- SW61 pad 2: COL0 -> COL1
- SW62 pad 2: COL1 -> COL2
- SW63 pad 2: COL1 -> COL3
- SW64 pad 2: COL2 -> COL4
- SW65 pad 2: COL2 -> COL5
- SW66 pad 2: COL3 -> COL6
- SW67 pad 2: COL3 -> COL7
- SW68 pad 2: COL4 -> COL8
- SW69 pad 2: COL4 -> COL9
- SW7 pad 2: COL3 -> COL6
- SW70 pad 2: COL5 -> COL10
- SW71 pad 2: COL5 -> COL11
- SW72 pad 1: Net-(D53-Pad2) -> Net-(D70-Pad2)
- SW72 pad 2: COL6 -> COL12
- SW73 pad 2: COL6 -> COL13
- SW74 pad 2: COL7 -> COL14
- SW75 pad 2: COL8 -> COL15
- SW76 pad 2: COL8 -> COL16
- SW77 pad 2: COL9 -> COL17
- SW8 pad 2: COL3 -> COL7
- SW80 pad 2: COL9 -> COL17
- SW82 pad 2: COL0 -> COL1
- SW83 pad 2: COL1 -> COL2
- SW84 pad 2: COL1 -> COL3
- SW85 pad 2: COL2 -> COL4
- SW86 pad 2: COL2 -> COL5
- SW87 pad 2: COL3 -> COL6
- SW88 pad 2: COL3 -> COL7
- SW89 pad 2: COL4 -> COL8
- SW9 pad 2: COL4 -> COL8
- SW90 pad 2: COL4 -> COL9
- SW91 pad 2: COL5 -> COL10
- SW92 pad 2: COL5 -> COL11
- SW93 pad 2: COL6 -> COL12
- SW94 pad 2: COL7 -> COL13
- SW95 pad 2: COL7 -> COL14
- SW96 pad 2: COL8 -> COL15
- SW97 pad 2: COL8 -> COL16
- SW98 pad 2: COL9 -> COL17
- U1 pad 1: COL9 -> unconnected-(U1-Pad1)
- U1 pad 10: VCC -> unconnected-(U1-Pad10)
- U1 pad 11: GND -> unconnected-(U1-Pad11)
- U1 pad 12: Net-(C5-Pad2) -> unconnected-(U1-Pad12)
- U1 pad 13: Net-(C4-Pad2) -> unconnected-(U1-Pad13)
- U1 pad 14: COL3 -> unconnected-(U1-Pad14)
- U1 pad 15: COL2 -> unconnected-(U1-Pad15)
- U1 pad 16: D+ -> unconnected-(U1-Pad16)
- U1 pad 17: D- -> unconnected-(U1-Pad17)
- U1 pad 18: BOOT -> unconnected-(U1-Pad18)
- U1 pad 19: COL1 -> unconnected-(U1-Pad19)
- U1 pad 2: COL8 -> unconnected-(U1-Pad2)
- U1 pad 20: COL0 -> unconnected-(U1-Pad20)
- U1 pad 21: COL4 -> unconnected-(U1-Pad21)
- U1 pad 22: ROW8 -> unconnected-(U1-Pad22)
- U1 pad 23: ROW7 -> unconnected-(U1-Pad23)
- U1 pad 24: ROW6 -> unconnected-(U1-Pad24)
- U1 pad 25: ROW5 -> unconnected-(U1-Pad25)
- U1 pad 26: ROW4 -> unconnected-(U1-Pad26)
- U1 pad 27: ROW3 -> unconnected-(U1-Pad27)
- U1 pad 28: ROW1 -> unconnected-(U1-Pad28)
- U1 pad 29: ROW0 -> unconnected-(U1-Pad29)
- U1 pad 3: COL7 -> unconnected-(U1-Pad3)
- U1 pad 30: VCC -> unconnected-(U1-Pad30)
- U1 pad 31: GND -> unconnected-(U1-Pad31)
- U1 pad 33: ROW2 -> unconnected-(U1-Pad33)
- U1 pad 34: ROW9 -> unconnected-(U1-Pad34)
- U1 pad 35: ROW10 -> unconnected-(U1-Pad35)
- U1 pad 36: ROW11 -> unconnected-(U1-Pad36)
- U1 pad 37: ROW12 -> unconnected-(U1-Pad37)
- U1 pad 4: COL6 -> unconnected-(U1-Pad4)
- U1 pad 5: COL5 -> unconnected-(U1-Pad5)
- U1 pad 6: MOSI -> unconnected-(U1-Pad6)
- U1 pad 7: MISO -> unconnected-(U1-Pad7)
- U1 pad 8: SCK -> unconnected-(U1-Pad8)
- U1 pad 9: RESET -> unconnected-(U1-Pad9)
Routing:
- added copper zone on B.Cu, net (none)
- added copper zone on F.Cu, net (none)
- removed copper zone on B.Cu, net GND
- removed copper zone on F.Cu, net GND
Other:
- board text added: "6U CENTER"
- board text added: "6U OFF 7U 10U"
- board text removed: "6U"
- board text removed: "6U OFF"
- board text removed: "7U&10U"

Commit message: Change footprint to 0xCB lib, add basic outline
Parts:
- added REF**: 2U Stabilizer, 0xcb:Stabilizer_Cherry_MX_2u, F.Cu at (465.1, 225.4)
- added REF**: 2U Stabilizer, 0xcb:Stabilizer_Cherry_MX_2u, F.Cu at (369.9, 196.8)
- added REF**: 2U Stabilizer, 0xcb:Stabilizer_Cherry_MX_2u, F.Cu at (124.6, 254.0)
- added REF**: 2U Stabilizer, 0xcb:Stabilizer_Cherry_MX_2u, F.Cu at (377.0, 225.4)
- added REF**: 2U Stabilizer, 0xcb:Stabilizer_Cherry_MX_2u, F.Cu at (465.1, 263.5)
- added REF**: 2U Stabilizer, 0xcb:Stabilizer_Cherry_MX_2u, F.Cu at (367.5, 234.9)
- U1: footprint BlackPill-STM32F401-temp:BlackPillSTM32F401CCU6 -> 0xcb:BlackPillSTM32F401CCU6
- moved D1 98.9 mm to (135.7, 169.9)
- moved D100 98.9 mm to (258.3, 169.9)
- moved D101 98.9 mm to (281.0, 172.2)
- moved D102 98.9 mm to (258.3, 172.2)
- moved D104 98.9 mm to (258.3, 184.2)
- moved D105 98.9 mm to (281.0, 184.2)
- moved D106 98.9 mm to (258.3, 181.8)
- moved D12 98.9 mm to (113.0, 181.8)
- moved D13 98.9 mm to (135.7, 172.2)
- moved D16 98.9 mm to (285.3, 181.8)
- moved D17 98.9 mm to (285.3, 184.2)
- moved D2 98.9 mm to (113.0, 169.9)
- moved D20 98.9 mm to (308.0, 181.8)
- moved D21 98.9 mm to (308.0, 184.2)
- moved D22 98.9 mm to (162.7, 184.2)
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Connections:
- SW107 pad 2: unconnected-(SW107-Pad2) -> COL12
Routing:
- removed copper zone on B.Cu, net (none)
- removed copper zone on F.Cu, net (none)
Other:
- board size 381 x 165.6 mm -> 412.8 x 147.6 mm
- board text removed: "2U STANDARD"

Commit message: Routing PCB, added extra layouts
Parts:
- removed D107: 1N4148, Diode_THT:D_DO-35_SOD27_P7.62mm_Horizontal
- removed REF** (x6): 2U Stabilizer, 0xcb:Stabilizer_Cherry_MX_2u
- added 2U Stabilizer: 2U Stabilizer, 0xcb:Stabilizer_Cherry_MX_2u, F.Cu at (124.6, 239.7)
- added 2U Stabilizer: 2U Stabilizer, 0xcb:Stabilizer_Cherry_MX_2u, F.Cu at (367.5, 220.7)
- added 2U Stabilizer: 2U Stabilizer, 0xcb:Stabilizer_Cherry_MX_2u, F.Cu at (272.3, 258.8)
- added 2U Stabilizer: 2U Stabilizer, 0xcb:Stabilizer_Cherry_MX_2u, F.Cu at (377.0, 211.1)
- added 2U Stabilizer: 2U Stabilizer, 0xcb:Stabilizer_Cherry_MX_2u, F.Cu at (205.6, 258.8)
- added 2U Stabilizer: 2U Stabilizer, 0xcb:Stabilizer_Cherry_MX_2u, F.Cu at (200.8, 258.8)
- added 2U Stabilizer: 2U Stabilizer, 0xcb:Stabilizer_Cherry_MX_2u, F.Cu at (267.5, 258.8)
- added 2U Stabilizer: 2U Stabilizer, 0xcb:Stabilizer_Cherry_MX_2u, F.Cu at (465.1, 249.2)
- added 2U Stabilizer: 2U Stabilizer, 0xcb:Stabilizer_Cherry_MX_2u, F.Cu at (369.9, 182.6)
- added 2U Stabilizer: 2U Stabilizer, 0xcb:Stabilizer_Cherry_MX_2u, F.Cu at (465.1, 211.1)
- added 6.25U Stabilizer: 6.25U Stabilizer, 0xcb:Stabilizer_Cherry_MX_6.25u, F.Cu at (234.2, 258.8)
- added 6U Stabilizer: 6U Stabilizer, 0xcb:Stabilizer_Cherry_MX_6u, F.Cu at (236.5, 258.8)
- added 7U Stabilizer: 7U Stabilizer, 0xcb:Stabilizer_Cherry_MX_7u, F.Cu at (227.0, 258.8)
- added 8U Stabilizer: 8U Stabilizer, 0xcb:Stabilizer_Cherry_MX_8u, F.Cu at (227.0, 258.8)
- added SW125: 1U, 0xcb:SW_Cherry_MX_PCB_1.00u, F.Cu at (241.3, 258.8)
- added SW126: 1U, 0xcb:SW_Cherry_MX_PCB_1.00u, F.Cu at (231.8, 258.8)
- SW100: value 1.25U GUI -> 1.25U ALT
- SW101: value 1.25U ALT -> 2.75U SPACE; footprint 0xcb:SW_Cherry_MX_PCB_1.25u -> 0xcb:SW_Cherry_MX_PCB_2.75u
- SW103: value 1U -> 2.25U SPACE; footprint 0xcb:SW_Cherry_MX_PCB_1.00u -> 0xcb:SW_Cherry_MX_PCB_2.25u
- SW113: value 1.5U CTRL -> 1.5U GUI
- SW114: value 1.5U GUI -> 1.5U CTRL
- SW116: value 7U -> 2.25U SPACE; footprint 0xcb:SW_Cherry_MX_PCB_7.00u -> 0xcb:SW_Cherry_MX_PCB_2.25u
- SW117: value 1.5U ALT -> 7U; footprint 0xcb:SW_Cherry_MX_PCB_1.50u -> 0xcb:SW_Cherry_MX_PCB_7.00u
- SW118: value 1.5U CTRL -> 2.75U SPACE; footprint 0xcb:SW_Cherry_MX_PCB_1.50u -> 0xcb:SW_Cherry_MX_PCB_2.75u
- SW119: value 1U -> 1.5U ALT; footprint 0xcb:SW_Cherry_MX_PCB_1.00u -> 0xcb:SW_Cherry_MX_PCB_1.50u
- SW120: value 1U -> 1.5U CTRL; footprint 0xcb:SW_Cherry_MX_PCB_1.00u -> 0xcb:SW_Cherry_MX_PCB_1.50u
- SW19, SW39: value 1U -> 2U; footprint 0xcb:SW_Cherry_MX_PCB_1.00u -> 0xcb:SW_Cherry_MX_PCB_2.00u
- SW35: value 2U -> 1U; footprint 0xcb:SW_Cherry_MX_PCB_2.00u -> 0xcb:SW_Cherry_MX_PCB_1.00u
- SW40: value 2U -> 1.5U; footprint 0xcb:SW_Cherry_MX_PCB_2.00u -> 0xcb:SW_Cherry_MX_PCB_1.50u
- SW41, SW54: value 1.5U -> 1U; footprint 0xcb:SW_Cherry_MX_PCB_1.50u -> 0xcb:SW_Cherry_MX_PCB_1.00u
- SW53: value 1U -> 1.5U; footprint 0xcb:SW_Cherry_MX_PCB_1.00u -> 0xcb:SW_Cherry_MX_PCB_1.50u
- SW58: value 1U -> ISO ENTER; footprint 0xcb:SW_Cherry_MX_PCB_1.00u -> 0xcb:SW_Cherry_MX_PCB_ISOEnter_Rotated90
- SW59: value ISO ENTER -> CAPSLOCK; footprint 0xcb:SW_Cherry_MX_PCB_ISOEnter_Rotated90 -> 0xcb:SW_Cherry_MX_PCB_1.75u
- SW60: value CAPSLOCK -> 1U; footprint 0xcb:SW_Cherry_MX_PCB_1.75u -> 0xcb:SW_Cherry_MX_PCB_1.00u
- SW71: value 1U -> ISO 1U
- SW72: value ISO 1U -> 2.25U; footprint 0xcb:SW_Cherry_MX_PCB_1.00u -> 0xcb:SW_Cherry_MX_PCB_2.25u
- SW73: value 2.25U -> 1U; footprint 0xcb:SW_Cherry_MX_PCB_2.25u -> 0xcb:SW_Cherry_MX_PCB_1.00u
- SW77: value 1U -> STEPPED; footprint 0xcb:SW_Cherry_MX_PCB_1.00u -> 0xcb:SW_Cherry_MX_PCB_1.25u
- SW78: value STEPPED -> 2.25U; footprint 0xcb:SW_Cherry_MX_PCB_1.25u -> 0xcb:SW_Cherry_MX_PCB_2.25u
- SW79: value 2.25U -> 2U; footprint 0xcb:SW_Cherry_MX_PCB_2.25u -> 0xcb:SW_Cherry_MX_PCB_2.00u
- SW80: value 2U -> ISO SHIFT; footprint 0xcb:SW_Cherry_MX_PCB_2.00u -> 0xcb:SW_Cherry_MX_PCB_1.25u
- SW81: value ISO SHIFT -> 1U; footprint 0xcb:SW_Cherry_MX_PCB_1.25u -> 0xcb:SW_Cherry_MX_PCB_1.00u
- SW92: value 1U -> 1.75U SHIFT; footprint 0xcb:SW_Cherry_MX_PCB_1.00u -> 0xcb:SW_Cherry_MX_PCB_1.75u
- SW93: value 1.75U SHIFT -> 1U; footprint 0xcb:SW_Cherry_MX_PCB_1.75u -> 0xcb:SW_Cherry_MX_PCB_1.00u
- SW98: value 1U -> 1.25U GUI; footprint 0xcb:SW_Cherry_MX_PCB_1.00u -> 0xcb:SW_Cherry_MX_PCB_1.25u
- moved SW80 350.9 mm to (115.1, 239.7), turned to 0 degrees
- moved SW77 350.3 mm to (115.1, 220.7)
- moved SW40 348.5 mm to (117.5, 201.6), turned to 0 degrees
- moved SW79 340.6 mm to (465.1, 249.2), turned to -90 degrees
- moved SW20 333.4 mm to (112.7, 182.6)
- moved SW21 333.4 mm to (131.8, 182.6)
- moved D35 328.2 mm to (439.2, 46.8)
- moved SW98 326.3 mm to (138.9, 258.8)
- moved D52 282.7 mm to (438.8, 36.2), turned to 0 degrees
- moved SW59 257.2 mm to (119.9, 220.7), turned to 0 degrees
- moved D74 227.7 mm to (117.5, 128.0), turned to -90 degrees
- moved D56 226.8 mm to (114.3, 129.5), turned to -90 degrees
- moved D96 225.9 mm to (449.6, 29.1), turned to 0 degrees
- moved D12 225.4 mm to (333.4, 134.3), turned to -90 degrees
- moved D13 218.4 mm to (349.2, 126.4), turned to -90 degrees
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Connections:
- D100 pad 1: ROW6 -> ROW5
- D101 pad 1: ROW6 -> ROW5
- D102 pad 1: ROW6 -> ROW5
- D103 pad 1: ROW6 -> ROW5
- D104 pad 1: ROW6 -> ROW5
- D105 pad 1: ROW6 -> ROW5
- D106 pad 1: ROW6 -> ROW5
- D18 pad 1: ROW1 -> ROW0
- D22 pad 1: ROW2 -> ROW1
- D23 pad 1: ROW2 -> ROW1
- D24 pad 1: ROW2 -> ROW1
- D25 pad 1: ROW2 -> ROW1
- D26 pad 1: ROW2 -> ROW1
- D27 pad 1: ROW2 -> ROW1
- D28 pad 1: ROW2 -> ROW1
- D29 pad 1: ROW2 -> ROW1
- D30 pad 1: ROW2 -> ROW1
- D31 pad 1: ROW2 -> ROW1
- D32 pad 1: ROW2 -> ROW1
- D33 pad 1: ROW2 -> ROW1
- D34 pad 1: ROW2 -> ROW1
- D35 pad 1: ROW2 -> ROW1
- D36 pad 1: ROW2 -> ROW1
- D37 pad 1: ROW2 -> ROW1
- D40 pad 1: ROW3 -> ROW2
- D41 pad 1: ROW3 -> ROW2
- D42 pad 1: ROW3 -> ROW2
- D43 pad 1: ROW3 -> ROW2
- D44 pad 1: ROW3 -> ROW2
- D45 pad 1: ROW3 -> ROW2
- D46 pad 1: ROW3 -> ROW2
- D47 pad 1: ROW3 -> ROW2
- D48 pad 1: ROW3 -> ROW2
- D49 pad 1: ROW3 -> ROW2
- D50 pad 1: ROW3 -> ROW2
- D51 pad 1: ROW3 -> ROW2
- D52 pad 1: ROW3 -> ROW2
- D53 pad 1: ROW3 -> ROW2
- D54 pad 1: ROW3 -> ROW2
- D55 pad 1: ROW3 -> ROW2
- D58 pad 1: ROW4 -> ROW3
- D59 pad 1: ROW4 -> ROW3
- D60 pad 1: ROW4 -> ROW3
- D61 pad 1: ROW4 -> ROW3
- D62 pad 1: ROW4 -> ROW3
- D63 pad 1: ROW4 -> ROW3
- D64 pad 1: ROW4 -> ROW3
- D65 pad 1: ROW4 -> ROW3
- D66 pad 1: ROW4 -> ROW3
- D67 pad 1: ROW4 -> ROW3
- D68 pad 1: ROW4 -> ROW3
- D69 pad 1: ROW4 -> ROW3
- D70 pad 1: ROW4 -> ROW3
- D71 pad 1: ROW4 -> ROW3
- D72 pad 1: ROW4 -> ROW3
- D73 pad 1: ROW4 -> ROW3
- D76 pad 1: ROW5 -> ROW4
- D77 pad 1: ROW5 -> ROW4
- D78 pad 1: ROW5 -> ROW4
- D79 pad 1: ROW5 -> ROW4
- D80 pad 1: ROW5 -> ROW4
- D81 pad 1: ROW5 -> ROW4
- D82 pad 1: ROW5 -> ROW4
- D83 pad 1: ROW5 -> ROW4
- D84 pad 1: ROW5 -> ROW4
- D85 pad 1: ROW5 -> ROW4
- D86 pad 1: ROW5 -> ROW4
- D87 pad 1: ROW5 -> ROW4
- D88 pad 1: ROW5 -> ROW4
- D89 pad 1: ROW5 -> ROW4
- D90 pad 1: ROW5 -> ROW4
- D91 pad 1: ROW5 -> ROW4
- D94 pad 1: ROW6 -> ROW5
- D95 pad 1: ROW6 -> ROW5
- D96 pad 1: ROW6 -> ROW5
- D97 pad 1: ROW6 -> ROW5
- D98 pad 1: ROW6 -> ROW5
- D99 pad 1: ROW6 -> ROW5
- SW10 pad 2: COL9 -> COL10
- SW100 pad 1: Net-(D105-Pad2) -> Net-(D103-Pad2)
- SW100 pad 2: COL1 -> COL2
- SW101 pad 1: Net-(D106-Pad2) -> Net-(D104-Pad2)
- SW101 pad 2: COL2 -> COL4
- SW102 pad 1: Net-(D107-Pad2) -> Net-(D106-Pad2)
- SW103 pad 1: Net-(D94-Pad2) -> Net-(D105-Pad2)
- SW104 pad 1: Net-(D102-Pad2) -> Net-(D99-Pad2)
- SW105 pad 1: Net-(D95-Pad2) -> Net-(D92-Pad2)
- SW106 pad 1: Net-(D103-Pad2) -> Net-(D100-Pad2)
- SW107 pad 1: Net-(D96-Pad2) -> Net-(D93-Pad2)
- SW107 pad 2: COL12 -> COL13
- SW108 pad 1: Net-(D97-Pad2) -> Net-(D94-Pad2)
- SW108 pad 2: COL13 -> COL14
- SW109 pad 1: Net-(D98-Pad2) -> Net-(D95-Pad2)
- SW109 pad 2: COL14 -> COL15
- SW11 pad 2: COL10 -> COL11
- SW110 pad 1: Net-(D99-Pad2) -> Net-(D96-Pad2)
- SW110 pad 2: COL15 -> COL16
- SW111 pad 1: Net-(D100-Pad2) -> Net-(D97-Pad2)
- SW111 pad 2: COL16 -> COL17
- SW112 pad 1: Net-(D101-Pad2) -> Net-(D98-Pad2)
- SW112 pad 2: COL17 -> COL18
- SW113 pad 1: Net-(D104-Pad2) -> Net-(D102-Pad2)
- SW113 pad 2: COL0 -> COL1
- SW114 pad 1: Net-(D105-Pad2) -> Net-(D101-Pad2)
- SW114 pad 2: COL1 -> COL0
- SW115 pad 1: Net-(D106-Pad2) -> Net-(D103-Pad2)
- SW116 pad 1: Net-(D107-Pad2) -> Net-(D104-Pad2)
- SW116 pad 2: COL6 -> COL4
- SW117 pad 1: Net-(D102-Pad2) -> Net-(D106-Pad2)
- SW117 pad 2: COL9 -> COL6
- SW118 pad 1: Net-(D103-Pad2) -> Net-(D105-Pad2)
- SW118 pad 2: COL11 -> COL8
- SW119 pad 1: Net-(D104-Pad2) -> Net-(D99-Pad2)
- SW119 pad 2: COL0 -> COL9
- SW12 pad 2: COL11 -> COL12
- SW120 pad 1: Net-(D105-Pad2) -> Net-(D100-Pad2)
- SW120 pad 2: COL1 -> COL11
- SW121 pad 1: Net-(D106-Pad2) -> Net-(D102-Pad2)
- SW121 pad 2: COL2 -> COL1
- SW122 pad 1: Net-(D107-Pad2) -> Net-(D106-Pad2)
- SW123 pad 1: Net-(D107-Pad2) -> Net-(D106-Pad2)
- SW124 pad 1: Net-(D107-Pad2) -> Net-(D106-Pad2)
- SW13 pad 2: COL12 -> COL13
- SW18 pad 2: COL14 -> COL18
- SW19 pad 1: Net-(D19-Pad2) -> Net-(D32-Pad2)
- SW19 pad 2: COL15 -> COL13
- SW2 pad 2: COL1 -> COL2
- SW20 pad 1: Net-(D20-Pad2) -> Net-(D19-Pad2)
- SW20 pad 2: COL16 -> COL0
- SW21 pad 1: Net-(D21-Pad2) -> Net-(D20-Pad2)
- SW21 pad 2: COL17 -> COL1
- SW22 pad 1: Net-(D22-Pad2) -> Net-(D21-Pad2)
- SW22 pad 2: COL0 -> COL2
- SW23 pad 1: Net-(D23-Pad2) -> Net-(D22-Pad2)
- SW23 pad 2: COL1 -> COL3
- SW24 pad 1: Net-(D24-Pad2) -> Net-(D23-Pad2)
- SW24 pad 2: COL2 -> COL4
- SW25 pad 1: Net-(D25-Pad2) -> Net-(D24-Pad2)
- SW25 pad 2: COL3 -> COL5
- SW26 pad 1: Net-(D26-Pad2) -> Net-(D25-Pad2)
- SW26 pad 2: COL4 -> COL6
- SW27 pad 1: Net-(D27-Pad2) -> Net-(D26-Pad2)
- SW27 pad 2: COL5 -> COL7
- SW28 pad 1: Net-(D28-Pad2) -> Net-(D27-Pad2)
- SW28 pad 2: COL6 -> COL8
- SW29 pad 1: Net-(D29-Pad2) -> Net-(D28-Pad2)
- SW29 pad 2: COL7 -> COL9
- SW3 pad 2: COL2 -> COL3
- SW30 pad 1: Net-(D30-Pad2) -> Net-(D29-Pad2)
- SW30 pad 2: COL8 -> COL10
- SW31 pad 1: Net-(D31-Pad2) -> Net-(D30-Pad2)
- SW31 pad 2: COL9 -> COL11
- SW32 pad 1: Net-(D32-Pad2) -> Net-(D31-Pad2)
- SW32 pad 2: COL10 -> COL12
- SW33 pad 1: Net-(D33-Pad2) -> Net-(D32-Pad2)
- SW33 pad 2: COL11 -> COL13
- SW34 pad 1: Net-(D34-Pad2) -> Net-(D33-Pad2)
- SW34 pad 2: COL12 -> COL14
- SW35 pad 1: Net-(D35-Pad2) -> Net-(D34-Pad2)
- SW35 pad 2: COL13 -> COL15
- SW36 pad 1: Net-(D36-Pad2) -> Net-(D35-Pad2)
- SW36 pad 2: COL14 -> COL16
- SW37 pad 1: Net-(D37-Pad2) -> Net-(D36-Pad2)
- SW37 pad 2: COL15 -> COL17
- SW38 pad 1: Net-(D38-Pad2) -> Net-(D37-Pad2)
- SW38 pad 2: COL16 -> COL18
- SW39 pad 1: Net-(D39-Pad2) -> Net-(D55-Pad2)
- SW39 pad 2: COL17 -> COL18
- SW4 pad 2: COL3 -> COL4
- SW40 pad 1: Net-(D57-Pad2) -> Net-(D38-Pad2)
- SW40 pad 2: COL17 -> COL0
- SW41 pad 1: Net-(D40-Pad2) -> Net-(D39-Pad2)
- SW41 pad 2: COL0 -> COL1
- SW42 pad 1: Net-(D41-Pad2) -> Net-(D40-Pad2)
- SW42 pad 2: COL1 -> COL2
- SW43 pad 1: Net-(D42-Pad2) -> Net-(D41-Pad2)
- SW43 pad 2: COL2 -> COL3
- SW44 pad 1: Net-(D43-Pad2) -> Net-(D42-Pad2)
- SW44 pad 2: COL3 -> COL4
- SW45 pad 1: Net-(D44-Pad2) -> Net-(D43-Pad2)
- SW45 pad 2: COL4 -> COL5
- SW46 pad 1: Net-(D45-Pad2) -> Net-(D44-Pad2)
- SW46 pad 2: COL5 -> COL6
- SW47 pad 1: Net-(D46-Pad2) -> Net-(D45-Pad2)
- SW47 pad 2: COL6 -> COL7
- SW48 pad 1: Net-(D47-Pad2) -> Net-(D46-Pad2)
- SW48 pad 2: COL7 -> COL8
- SW49 pad 1: Net-(D48-Pad2) -> Net-(D47-Pad2)
- SW49 pad 2: COL8 -> COL9
- SW5 pad 2: COL4 -> COL5
- SW50 pad 1: Net-(D49-Pad2) -> Net-(D48-Pad2)
- SW50 pad 2: COL9 -> COL10
- SW51 pad 1: Net-(D50-Pad2) -> Net-(D49-Pad2)
- SW51 pad 2: COL10 -> COL11
- SW52 pad 1: Net-(D51-Pad2) -> Net-(D50-Pad2)
- SW52 pad 2: COL11 -> COL12
- SW53 pad 1: Net-(D52-Pad2) -> Net-(D51-Pad2)
- SW53 pad 2: COL12 -> COL13
- SW54 pad 1: Net-(D53-Pad2) -> Net-(D52-Pad2)
- SW54 pad 2: COL13 -> COL15
- SW55 pad 1: Net-(D54-Pad2) -> Net-(D53-Pad2)
- SW55 pad 2: COL14 -> COL16
- SW56 pad 1: Net-(D55-Pad2) -> Net-(D54-Pad2)
- SW56 pad 2: COL15 -> COL17
- SW57 pad 1: Net-(D56-Pad2) -> Net-(D55-Pad2)
- SW57 pad 2: COL16 -> COL18
- SW58 pad 1: Net-(D57-Pad2) -> Net-(D69-Pad2)
- SW58 pad 2: COL17 -> COL13
- SW59 pad 1: Net-(D71-Pad2) -> Net-(D56-Pad2)
- SW59 pad 2: COL13 -> COL0
- SW6 pad 2: COL5 -> COL6
- SW60 pad 1: Net-(D58-Pad2) -> Net-(D57-Pad2)
- SW60 pad 2: COL0 -> COL1
- SW61 pad 1: Net-(D59-Pad2) -> Net-(D58-Pad2)
- SW61 pad 2: COL1 -> COL2
- SW62 pad 1: Net-(D60-Pad2) -> Net-(D59-Pad2)
- SW62 pad 2: COL2 -> COL3
- SW63 pad 1: Net-(D61-Pad2) -> Net-(D60-Pad2)
- SW63 pad 2: COL3 -> COL4
- SW64 pad 1: Net-(D62-Pad2) -> Net-(D61-Pad2)
- SW64 pad 2: COL4 -> COL5
- SW65 pad 1: Net-(D63-Pad2) -> Net-(D62-Pad2)
- SW65 pad 2: COL5 -> COL6
- SW66 pad 1: Net-(D64-Pad2) -> Net-(D63-Pad2)
- SW66 pad 2: COL6 -> COL7
- SW67 pad 1: Net-(D65-Pad2) -> Net-(D64-Pad2)
- SW67 pad 2: COL7 -> COL8
- SW68 pad 1: Net-(D66-Pad2) -> Net-(D65-Pad2)
- SW68 pad 2: COL8 -> COL9
- SW69 pad 1: Net-(D67-Pad2) -> Net-(D66-Pad2)
- SW69 pad 2: COL9 -> COL10
- SW7 pad 2: COL6 -> COL7
- SW70 pad 1: Net-(D68-Pad2) -> Net-(D67-Pad2)
- SW70 pad 2: COL10 -> COL11
- SW71 pad 1: Net-(D69-Pad2) -> Net-(D68-Pad2)
- SW71 pad 2: COL11 -> COL12
- SW72 pad 1: Net-(D70-Pad2) -> Net-(D69-Pad2)
- SW72 pad 2: COL12 -> COL13
- SW73 pad 1: Net-(D71-Pad2) -> Net-(D70-Pad2)
- SW73 pad 2: COL13 -> COL15
- SW74 pad 1: Net-(D72-Pad2) -> Net-(D71-Pad2)
- SW74 pad 2: COL14 -> COL16
- SW75 pad 1: Net-(D73-Pad2) -> Net-(D72-Pad2)
- SW75 pad 2: COL15 -> COL17
- SW76 pad 1: Net-(D74-Pad2) -> Net-(D73-Pad2)
- SW76 pad 2: COL16 -> COL18
- SW77 pad 1: Net-(D75-Pad2) -> Net-(D56-Pad2)
- SW77 pad 2: COL17 -> COL0
- SW78 pad 1: Net-(D58-Pad2) -> Net-(D74-Pad2)
- SW79 pad 1: Net-(D76-Pad2) -> Net-(D91-Pad2)
- SW79 pad 2: COL0 -> COL18
- SW8 pad 2: COL7 -> COL8
- SW80 pad 1: Net-(D93-Pad2) -> Net-(D74-Pad2)
- SW80 pad 2: COL17 -> COL0
- SW81 pad 1: Net-(D76-Pad2) -> Net-(D75-Pad2)
- SW81 pad 2: COL0 -> COL1
- SW82 pad 1: Net-(D77-Pad2) -> Net-(D76-Pad2)
- SW82 pad 2: COL1 -> COL2
- SW83 pad 1: Net-(D78-Pad2) -> Net-(D77-Pad2)
- SW83 pad 2: COL2 -> COL3
- SW84 pad 1: Net-(D79-Pad2) -> Net-(D78-Pad2)
- SW84 pad 2: COL3 -> COL4
- SW85 pad 1: Net-(D80-Pad2) -> Net-(D79-Pad2)
- SW85 pad 2: COL4 -> COL5
- SW86 pad 1: Net-(D81-Pad2) -> Net-(D80-Pad2)
- SW86 pad 2: COL5 -> COL6
- SW87 pad 1: Net-(D82-Pad2) -> Net-(D81-Pad2)
- SW87 pad 2: COL6 -> COL7
- SW88 pad 1: Net-(D83-Pad2) -> Net-(D82-Pad2)
- SW88 pad 2: COL7 -> COL8
- SW89 pad 1: Net-(D84-Pad2) -> Net-(D83-Pad2)
- SW89 pad 2: COL8 -> COL9
- SW9 pad 2: COL8 -> COL9
- SW90 pad 1: Net-(D85-Pad2) -> Net-(D84-Pad2)
- SW90 pad 2: COL9 -> COL10
- SW91 pad 1: Net-(D86-Pad2) -> Net-(D85-Pad2)
- SW91 pad 2: COL10 -> COL11
- SW92 pad 1: Net-(D87-Pad2) -> Net-(D86-Pad2)
- SW92 pad 2: COL11 -> COL12
- SW93 pad 1: Net-(D88-Pad2) -> Net-(D87-Pad2)
- SW93 pad 2: COL12 -> COL14
- SW94 pad 1: Net-(D89-Pad2) -> Net-(D88-Pad2)
- SW94 pad 2: COL13 -> COL15
- SW95 pad 1: Net-(D90-Pad2) -> Net-(D89-Pad2)
- SW95 pad 2: COL14 -> COL16
- SW96 pad 1: Net-(D91-Pad2) -> Net-(D90-Pad2)
- SW96 pad 2: COL15 -> COL17
- SW97 pad 1: Net-(D92-Pad2) -> Net-(D91-Pad2)
- SW97 pad 2: COL16 -> COL18
- SW98 pad 1: Net-(D93-Pad2) -> Net-(D102-Pad2)
- SW98 pad 2: COL17 -> COL1
- SW99 pad 1: Net-(D104-Pad2) -> Net-(D101-Pad2)
Routing:
- net Net-(D106-Pad2): track 0.00 -> 159.8 mm
- net Net-(D104-Pad2): track 0.00 -> 147.9 mm
- net Net-(D94-Pad2): track 0.00 -> 143.9 mm
- net Net-(D93-Pad2): track 0.00 -> 142.2 mm
- net Net-(D99-Pad2): track 0.00 -> 140.3 mm
- net Net-(D101-Pad2): track 0.00 -> 139.7 mm
- net Net-(D105-Pad2): track 0.00 -> 138.1 mm
- net Net-(D100-Pad2): track 0.00 -> 136.6 mm
- net Net-(D92-Pad2): track 0.00 -> 135.2 mm
- net Net-(D103-Pad2): track 0.00 -> 132.8 mm
- net Net-(D102-Pad2): track 0.00 -> 127.1 mm
- net Net-(D87-Pad2): track 0.00 -> 121.4 mm
- net Net-(D80-Pad2): track 0.00 -> 117.6 mm
- net Net-(D81-Pad2): track 0.00 -> 117.0 mm
- net Net-(D74-Pad2): track 0.00 -> 116.0 mm
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Other:
- board size 412.8 x 147.6 mm -> 412.8 x 133.3 mm
- board text removed: "1.25U"
- board text removed: "1.5U"
- board text removed: "1U"
- board text removed: "1U ISO"
- board text removed: "2.25U"
- board text removed: "6.25U"
- board text removed: "6U CENTER"
- board text removed: "6U OFF 7U 10U"
- board text removed: "ANSI ENTER"
- board text removed: "I PAID FOR THE ENTIRE SET, SO I AM GOING TO USE THE ENTIRE SET"
- board text removed: "ISO"
- board text removed: "ISO ENTER"
- board text removed: "STANDARD"
- board text removed: "STEPPED"
